File: lab4/exercise1/exercise1.kicad_sch (KiCad schematic)
At the start: 6 parts, among them SW1 SW_SPDT

Commit message: did kicad things
Parts:
- C1: footprint (none) -> C_Radial_D5.0mm_H5.0mm_P2.00mm
- D1: footprint (none) -> LED_D5.0mm
- R1, R2: footprint (none) -> R_Axial_DIN0516_L15.5mm_D5.0mm_P20.32mm_Horizontal
- SW1: footprint (none) -> SW_E-Switch_EG1224_SPDT_Angled
- V1: footprint (none) -> JST_PH_B2B-PH-K_1x02_P2.00mm_Vertical
Changed lines of the file:
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@@
   (symbol (lib_id "Device:LED") (at 125.73 96.52 90) (unit 1)
     (in_bom yes) (on_board yes) (fields_autoplaced)
-    (property "Reference" "D1" (id 0) (at 129.54 96.8374 90)
+    (property "Reference" "D1" (id 0) (at 129.54 98.1074 90)
       (effects (font (size 1.27 1.27)) (justify right))
     )
@@
       (effects (font (size 1.27 1.27)) (justify right) hide)
     )
-    (property "Footprint" "" (id 2) (at 125.73 96.52 0)
+    (property "Footprint" "LED_D5.0mm" (id 2) (at 125.73 96.52 0)
       (effects (font (size 1.27 1.27)) hide)
     )
@@
     (property "Reference" "R1" (id 0) (at 77.47 74.93 90))
     (property "Value" "2.2 kOhms" (id 1) (at 77.47 77.47 90))
-    (property "Footprint" "" (id 2) (at 77.47 83.058 90)
+    (property "Footprint" "R_Axial_DIN0516_L15.5mm_D5.0mm_P20.32mm_Horizontal" (id 2) (at 77.47 83.058 90)
       (effects (font (size 1.27 1.27)) hide)
     )
@@
   (symbol (lib_id "Switch:SW_SPDT") (at 91.44 81.28 0) (unit 1)
     (in_bom yes) (on_board yes) (fields_autoplaced)
-    (property "Reference" "SW1" (id 0) (at 91.44 73.66 0))
+    (property "Reference" "SW1" (id 0) (at 91.44 76.2 0))
     (property "Value" "SW_SPDT" (id 1) (at 91.44 76.2 0)
       (effects (font (size 1.27 1.27)) hide)
     )
-    (property "Footprint" "" (id 2) (at 91.44 81.28 0)
+    (property "Footprint" "SW_E-Switch_EG1224_SPDT_Angled" (id 2) (at 91.44 81.28 0)
       (effects (font (size 1.27 1.27)) hide)
     )
@@
     (property "Reference" "V1" (id 0) (at 66.675 82.55 0))
     (property "Value" "9 V" (id 1) (at 66.675 85.09 0))
-    (property "Footprint" "" (id 2) (at 66.04 87.63 0)
+    (property "Footprint" "JST_PH_B2B-PH-K_1x02_P2.00mm_Vertical" (id 2) (at 66.04 87.63 0)
       (effects (font (size 1.27 1.27)) hide)
     )
@@
       (effects (font (size 1.27 1.27)) (justify left))
     )
-    (property "Footprint" "" (id 2) (at 105.1052 95.25 0)
+    (property "Footprint" "C_Radial_D5.0mm_H5.0mm_P2.00mm" (id 2) (at 105.1052 95.25 0)
       (effects (font (size 1.27 1.27)) hide)
     )
@@
       (effects (font (size 1.27 1.27)) (justify left))
     )
-    (property "Footprint" "" (id 2) (at 123.952 87.63 90)
+    (property "Footprint" "R_Axial_DIN0516_L15.5mm_D5.0mm_P20.32mm_Horizontal" (id 2) (at 123.952 87.63 90)
       (effects (font (size 1.27 1.27)) hide)
     )
@@
   (symbol_instances
     (path "/c40bc5fb-458a-4663-a2c4-834a5235dba4"
-      (reference "C1") (unit 1) (value "4.7 microF") (footprint "")
+      (reference "C1") (unit 1) (value "4.7 microF") (footprint "C_Radial_D5.0mm_H5.0mm_P2.00mm")
     )
     (path "/0f2263f9-3aae-45dd-8cef-66d71a2f7da9"
-      (reference "D1") (unit 1) (value "LED") (footprint "")
+      (reference "D1") (unit 1) (value "LED") (footprint "LED_D5.0mm")
     )
     (path "/108577e2-276f-484b-9356-c66c21d3e106"
-      (reference "R1") (unit 1) (value "2.2 kOhms") (footprint "")
+      (reference "R1") (unit 1) (value "2.2 kOhms") (footprint "R_Axial_DIN0516_L15.5mm_D5.0mm_P20.32mm_Horizontal")
     )
     (path "/e394a2c2-9c73-45ec-9d14-1aa89064ba11"
-      (reference "R2") (unit 1) (value "20 kOhms") (footprint "")
+      (reference "R2") (unit 1) (value "20 kOhms") (footprint "R_Axial_DIN0516_L15.5mm_D5.0mm_P20.32mm_Horizontal")
     )
     (path "/3a9b2c98-fd5b-4b37-934d-f49cbe57125f"
-      (reference "SW1") (unit 1) (value "SW_SPDT") (footprint "")
+      (reference "SW1") (unit 1) (value "SW_SPDT") (footprint "SW_E-Switch_EG1224_SPDT_Angled")
     )
     (path "/5cf5e501-1f0c-4391-82f3-eb6867bd5797"
-      (reference "V1") (unit 1) (value "9 V") (footprint "")
+      (reference "V1") (unit 1) (value "9 V") (footprint "JST_PH_B2B-PH-K_1x02_P2.00mm_Vertical")
     )
   )
