File: lab4/exercise2/exercise2.kicad_sch (KiCad schematic)
At the start: 10 parts, among them J1 Conn_01x02_Male, U1 NE555D

Commit message: did kicad things
Parts:
- C1: footprint (none) -> CP_EIA-3216-18_Kemet-A_Pad1.58x1.35mm_HandSolder
- C2: footprint (none) -> C_0805_2012Metric_Pad1.18x1.45mm_HandSolder
- D1, D2: footprint (none) -> LED_1206_3216Metric_Pad1.42x1.75mm_HandSolder
- J1: footprint (none) -> TerminalBlock_bornier-2_P5.08mm
- R1, R2, R3, R4: footprint (none) -> R_0805_2012Metric_Pad1.20x1.40mm_HandSolder
- U1: footprint Package_SO:SOIC-8_3.9x4.9mm_P1.27mm -> SOIC-8-1EP_3.9x4.9mm_P1.27mm_EP2.29x3mm
Changed lines of the file:
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@@
       (effects (font (size 1.27 1.27)) (justify left))
     )
-    (property "Footprint" "" (id 2) (at 85.852 80.01 90)
+    (property "Footprint" "R_0805_2012Metric_Pad1.20x1.40mm_HandSolder" (id 2) (at 85.852 80.01 90)
       (effects (font (size 1.27 1.27)) hide)
     )
@@
   (symbol (lib_id "Connector:Conn_01x02_Male") (at 137.16 54.61 90) (unit 1)
     (in_bom yes) (on_board yes) (fields_autoplaced)
-    (property "Reference" "J1" (id 0) (at 140.97 52.7049 90)
+    (property "Reference" "J1" (id 0) (at 140.97 53.9749 90)
       (effects (font (size 1.27 1.27)) (justify right))
     )
@@
       (effects (font (size 1.27 1.27)) (justify right) hide)
     )
-    (property "Footprint" "" (id 2) (at 137.16 54.61 0)
+    (property "Footprint" "TerminalBlock_bornier-2_P5.08mm" (id 2) (at 137.16 54.61 0)
       (effects (font (size 1.27 1.27)) hide)
     )
@@
       (effects (font (size 1.27 1.27)) (justify left))
     )
-    (property "Footprint" "Package_SO:SOIC-8_3.9x4.9mm_P1.27mm" (id 2) (at 163.83 111.76 0)
+    (property "Footprint" "SOIC-8-1EP_3.9x4.9mm_P1.27mm_EP2.29x3mm" (id 2) (at 163.83 111.76 0)
       (effects (font (size 1.27 1.27)) hide)
     )
@@
       (effects (font (size 1.27 1.27)) (justify left))
     )
-    (property "Footprint" "" (id 2) (at 88.5952 138.43 0)
+    (property "Footprint" "CP_EIA-3216-18_Kemet-A_Pad1.58x1.35mm_HandSolder" (id 2) (at 88.5952 138.43 0)
       (effects (font (size 1.27 1.27)) hide)
     )
@@
       (effects (font (size 1.27 1.27)) (justify left))
     )
-    (property "Footprint" "" (id 2) (at 85.852 106.68 90)
+    (property "Footprint" "R_0805_2012Metric_Pad1.20x1.40mm_HandSolder" (id 2) (at 85.852 106.68 90)
       (effects (font (size 1.27 1.27)) hide)
     )
@@
       (effects (font (size 1.27 1.27)) (justify right))
     )
-    (property "Footprint" "" (id 2) (at 190.5 69.85 0)
+    (property "Footprint" "LED_1206_3216Metric_Pad1.42x1.75mm_HandSolder" (id 2) (at 190.5 69.85 0)
       (effects (font (size 1.27 1.27)) hide)
     )
@@
       (effects (font (size 1.27 1.27)) (justify left))
     )
-    (property "Footprint" "" (id 2) (at 188.722 90.17 90)
+    (property "Footprint" "R_0805_2012Metric_Pad1.20x1.40mm_HandSolder" (id 2) (at 188.722 90.17 90)
       (effects (font (size 1.27 1.27)) hide)
     )
@@
       (effects (font (size 1.27 1.27)) (justify left))
     )
-    (property "Footprint" "" (id 2) (at 113.9952 124.46 0)
+    (property "Footprint" "C_0805_2012Metric_Pad1.18x1.45mm_HandSolder" (id 2) (at 113.9952 124.46 0)
       (effects (font (size 1.27 1.27)) hide)
     )
@@
       (effects (font (size 1.27 1.27)) (justify left))
     )
-    (property "Footprint" "" (id 2) (at 188.722 109.22 90)
+    (property "Footprint" "R_0805_2012Metric_Pad1.20x1.40mm_HandSolder" (id 2) (at 188.722 109.22 90)
       (effects (font (size 1.27 1.27)) hide)
     )
@@
       (effects (font (size 1.27 1.27)) (justify right))
     )
-    (property "Footprint" "" (id 2) (at 190.5 129.54 0)
+    (property "Footprint" "LED_1206_3216Metric_Pad1.42x1.75mm_HandSolder" (id 2) (at 190.5 129.54 0)
       (effects (font (size 1.27 1.27)) hide)
     )
@@
     )
     (path "/46c9af93-c70f-4113-8a50-a4bcf012a794"
-      (reference "C1") (unit 1) (value "10 microF") (footprint "")
+      (reference "C1") (unit 1) (value "10 microF") (footprint "CP_EIA-3216-18_Kemet-A_Pad1.58x1.35mm_HandSolder")
     )
     (path "/ccc9e679-a1d8-4fe2-85fe-82e8190a47ed"
-      (reference "C2") (unit 1) (value "0.01 microF") (footprint "")
+      (reference "C2") (unit 1) (value "0.01 microF") (footprint "C_0805_2012Metric_Pad1.18x1.45mm_HandSolder")
     )
     (path "/869e40e3-43ed-46fd-9288-4c7727e2964f"
-      (reference "D1") (unit 1) (value "LED") (footprint "")
+      (reference "D1") (unit 1) (value "LED") (footprint "LED_1206_3216Metric_Pad1.42x1.75mm_HandSolder")
     )
     (path "/fc3b3f85-fbe9-4173-9ee6-8776ee178866"
-      (reference "D2") (unit 1) (value "LED") (footprint "")
+      (reference "D2") (unit 1) (value "LED") (footprint "LED_1206_3216Metric_Pad1.42x1.75mm_HandSolder")
     )
     (path "/0c2d70d0-a595-4788-888c-e46e88562f78"
-      (reference "J1") (unit 1) (value "Conn_01x02_Male") (footprint "")
+      (reference "J1") (unit 1) (value "Conn_01x02_Male") (footprint "TerminalBlock_bornier-2_P5.08mm")
     )
     (path "/09cd902a-5694-40f8-aa6c-0389a4d0f8b7"
-      (reference "R1") (unit 1) (value "1k") (footprint "")
+      (reference "R1") (unit 1) (value "1k") (footprint "R_0805_2012Metric_Pad1.20x1.40mm_HandSolder")
     )
     (path "/585f1182-f528-453f-9d90-070c9499fea5"
-      (reference "R2") (unit 1) (value "10k") (footprint "")
+      (reference "R2") (unit 1) (value "10k") (footprint "R_0805_2012Metric_Pad1.20x1.40mm_HandSolder")
     )
     (path "/adf691f1-4e0e-4463-9458-b3a98d956f85"
-      (reference "R3") (unit 1) (value "1k") (footprint "")
+      (reference "R3") (unit 1) (value "1k") (footprint "R_0805_2012Metric_Pad1.20x1.40mm_HandSolder")
     )
     (path "/e80c4582-61d0-478b-afde-e8e5a2e669a5"
-      (reference "R4") (unit 1) (value "1k") (footprint "")
+      (reference "R4") (unit 1) (value "1k") (footprint "R_0805_2012Metric_Pad1.20x1.40mm_HandSolder")
     )
     (path "/2a036ac8-c1a6-41e5-833d-ca9dcb7db1ab"
-      (reference "U1") (unit 1) (value "NE555D") (footprint "Package_SO:SOIC-8_3.9x4.9mm_P1.27mm")
-    )
-  )
+      (reference "U1") (unit 1) (value "NE555D") (footprint "SOIC-8-1EP_3.9x4.9mm_P1.27mm_EP2.29x3mm")
+    )
+  )
